File: Main.brd (EAGLE design)
At the start: 99.6 x 43.2 mm, 44 parts, among them U1 74HC595D-SOIC16, X1 87758-0816

Commit message: BugFix
Connections:
- removed net N$35: U$1.8, X1.7
- removed net N$36: U$1.9, X1.8
- new net NRF_CE: U$1.27, U$2.CE
- net +5V: now also X1.7
- net GND: now also X1.8
Routing:
- net NRF_CE: track 0.00 -> 30.1 mm
- net N$35: track 7.33 -> 0.00 mm
- net N$36: track 5.00 -> 0.00 mm
- net +5V: track 172.9 -> 176.3 mm
Changed lines of the file:
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@@
 <grid distance="0.2" unitdist="mm" unit="mm" style="dots" multiple="1" display="yes" altdistance="0.01" altunitdist="mm" altunit="mm"/>
 <layers>
-<layer number="1" name="Top" color="4" fill="1" visible="no" active="yes"/>
+<layer number="1" name="Top" color="4" fill="1" visible="yes" active="yes"/>
 <layer number="2" name="Route2" color="1" fill="3" visible="no" active="no"/>
 <layer number="3" name="Route3" color="4" fill="3" visible="no" active="no"/>
@@
 <layer number="14" name="Route14" color="1" fill="6" visible="no" active="no"/>
 <layer number="15" name="Route15" color="4" fill="6" visible="no" active="no"/>
-<layer number="16" name="Bottom" color="1" fill="1" visible="no" active="yes"/>
-<layer number="17" name="Pads" color="2" fill="1" visible="no" active="yes"/>
-<layer number="18" name="Vias" color="2" fill="1" visible="no" active="yes"/>
+<layer number="16" name="Bottom" color="1" fill="1" visible="yes" active="yes"/>
+<layer number="17" name="Pads" color="2" fill="1" visible="yes" active="yes"/>
+<layer number="18" name="Vias" color="2" fill="1" visible="yes" active="yes"/>
 <layer number="19" name="Unrouted" color="6" fill="1" visible="yes" active="yes"/>
 <layer number="20" name="Dimension" color="15" fill="1" visible="yes" active="yes"/>
-<layer number="21" name="tPlace" color="7" fill="1" visible="no" active="yes"/>
+<layer number="21" name="tPlace" color="7" fill="1" visible="yes" active="yes"/>
 <layer number="22" name="bPlace" color="7" fill="1" visible="no" active="yes"/>
 <layer number="23" name="tOrigins" color="15" fill="1" visible="no" active="yes"/>
@@
 <layer number="27" name="tValues" color="7" fill="1" visible="no" active="yes"/>
 <layer number="28" name="bValues" color="7" fill="1" visible="no" active="yes"/>
-<layer number="29" name="tStop" color="7" fill="3" visible="no" active="yes"/>
+<layer number="29" name="tStop" color="7" fill="3" visible="yes" active="yes"/>
 <layer number="30" name="bStop" color="7" fill="6" visible="no" active="yes"/>
 <layer number="31" name="tCream" color="7" fill="4" visible="no" active="yes"/>
@@
 <via x="42.2" y="26.6" extent="1-16" drill="0.4" diameter="1.27"/>
 <via x="59.8" y="6.8" extent="1-16" drill="0.4" diameter="1.27"/>
-<via x="45" y="31" extent="1-16" drill="0.4" diameter="1.27"/>
+<via x="50.8" y="30.6" extent="1-16" drill="0.4" diameter="1.27"/>
+<contactref element="X1" pad="8"/>
+<via x="67" y="40.8" extent="1-16" drill="0.4" diameter="1.27"/>
+<via x="77.8" y="20.2" extent="1-16" drill="0.4" diameter="1.27"/>
 </signal>
 <signal name="N$1">
@@
 <wire x1="20" y1="7.6" x2="16.4" y2="11.2" width="0.4064" layer="16"/>
 <wire x1="16.4" y1="11.2" x2="16.4" y2="20.6" width="0.4064" layer="16"/>
+<contactref element="X1" pad="7"/>
+<wire x1="23.6" y1="29.8" x2="22.919" y2="29.8" width="0.4064" layer="16"/>
+<wire x1="22.919" y1="29.8" x2="20.979" y2="27.86" width="0.4064" layer="16"/>
 </signal>
 <signal name="+3V3">
@@
 <wire x1="28.8" y1="31.8" x2="25.6" y2="31.8" width="0.25" layer="1"/>
 </signal>
-<signal name="N$35">
-<contactref element="U$1" pad="8"/>
-<contactref element="X1" pad="7"/>
-<wire x1="30.48" y1="30.89" x2="27.29" y2="30.89" width="0.25" layer="1"/>
-<wire x1="27.29" y1="30.89" x2="27.2" y2="30.8" width="0.25" layer="1"/>
-<wire x1="27.2" y1="30.8" x2="24.6" y2="30.8" width="0.25" layer="1"/>
-<wire x1="24.6" y1="30.8" x2="23.6" y2="29.8" width="0.25" layer="1"/>
-</signal>
-<signal name="N$36">
-<contactref element="U$1" pad="9"/>
-<contactref element="X1" pad="8"/>
-<wire x1="30.48" y1="30.09" x2="27.29" y2="30.09" width="0.25" layer="1"/>
-<wire x1="27.29" y1="30.09" x2="27" y2="29.8" width="0.25" layer="1"/>
-<wire x1="27" y1="29.8" x2="25.6" y2="29.8" width="0.25" layer="1"/>
-</signal>
 <signal name="N$37">
 <via x="89" y="6.6" extent="1-16" drill="4.2" diameter="12"/>
@@
 <wire x1="88.25" y1="13.8" x2="90.75" y2="13.8" width="0.4064" layer="1"/>
 </signal>
+<signal name="NRF_CE">
+<contactref element="U$2" pad="CE"/>
+<contactref element="U$1" pad="27"/>
+<wire x1="42.08" y1="31.69" x2="50.29" y2="31.69" width="0.4064" layer="1"/>
+<wire x1="50.29" y1="31.69" x2="56.2" y2="37.6" width="0.4064" layer="1"/>
+<wire x1="56.2" y1="37.6" x2="58.8" y2="37.6" width="0.4064" layer="1"/>
+<wire x1="58.8" y1="37.6" x2="59.2" y2="37.2" width="0.4064" layer="1"/>
+<wire x1="59.2" y1="37.2" x2="59.2" y2="32.4" width="0.4064" layer="1"/>
+<wire x1="59.2" y1="32.4" x2="60" y2="31.6" width="0.4064" layer="1"/>
+<wire x1="60" y1="31.6" x2="62.66" y2="31.6" width="0.254" layer="1"/>
+<wire x1="62.66" y1="31.6" x2="63.93" y2="30.33" width="0.254" layer="1"/>
+</signal>
 </signals>
