File: Main.sch (EAGLE design)
At the start: 44 parts, among them U1 74HC595D-SOIC16, X1 87758-0816

Commit message: BugFix
Connections:
- removed net N$35: U$1.8, X1-7.S
- removed net N$36: U$1.9, X1-8.S
- new net NRF_CE: U$1.27, U$2.CE
- net +5V: now also X1-7.S
- net GND: now also X1-8.S
Changed lines of the file:
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@@
 <part name="R17" library="rcl" deviceset="R-EU_" device="M0805"/>
 <part name="LED2" library="led" deviceset="LED" device="CHIP-LED0805"/>
+<part name="P+3" library="supply1" deviceset="+5V" device=""/>
+<part name="GND3" library="supply1" deviceset="GND" device=""/>
 </parts>
 <sheets>
@@
 <instance part="R17" gate="G$1" x="121.92" y="104.14" rot="R180"/>
 <instance part="LED2" gate="G$1" x="121.92" y="96.52" rot="R270"/>
+<instance part="P+3" gate="1" x="-106.68" y="-25.4" rot="R90"/>
+<instance part="GND3" gate="1" x="-86.36" y="-27.94"/>
 </instances>
 <busses>
@@
 <label x="7.62" y="38.1" size="1.778" layer="95" rot="R90"/>
 </segment>
+<segment>
+<pinref part="X1" gate="-8" pin="S"/>
+<pinref part="GND3" gate="1" pin="GND"/>
+<wire x1="-81.28" y1="-25.4" x2="-86.36" y2="-25.4" width="0.1524" layer="91"/>
+</segment>
 </net>
 <net name="N$1" class="0">
@@
 <wire x1="10.16" y1="48.26" x2="10.16" y2="33.02" width="0.1524" layer="91"/>
 <label x="10.16" y="38.1" size="1.778" layer="95" rot="R90"/>
+</segment>
+<segment>
+<pinref part="X1" gate="-7" pin="S"/>
+<pinref part="P+3" gate="1" pin="+5V"/>
+<wire x1="-101.6" y1="-25.4" x2="-104.14" y2="-25.4" width="0.1524" layer="91"/>
 </segment>
 </net>
@@
 </segment>
 </net>
-<net name="N$35" class="0">
-<segment>
-<pinref part="U$1" gate="G$1" pin="8"/>
-<wire x1="-33.02" y1="-5.08" x2="-109.22" y2="-5.08" width="0.1524" layer="91"/>
-<wire x1="-109.22" y1="-5.08" x2="-109.22" y2="-25.4" width="0.1524" layer="91"/>
-<pinref part="X1" gate="-7" pin="S"/>
-<wire x1="-109.22" y1="-25.4" x2="-101.6" y2="-25.4" width="0.1524" layer="91"/>
-</segment>
-</net>
-<net name="N$36" class="0">
-<segment>
-<pinref part="U$1" gate="G$1" pin="9"/>
-<wire x1="-33.02" y1="-7.62" x2="-88.9" y2="-7.62" width="0.1524" layer="91"/>
-<wire x1="-88.9" y1="-7.62" x2="-88.9" y2="-25.4" width="0.1524" layer="91"/>
-<pinref part="X1" gate="-8" pin="S"/>
-<wire x1="-88.9" y1="-25.4" x2="-81.28" y2="-25.4" width="0.1524" layer="91"/>
-</segment>
-</net>
 <net name="N$4" class="0">
 <segment>
@@
 </segment>
 </net>
+<net name="NRF_CE" class="0">
+<segment>
+<pinref part="U$2" gate="G$1" pin="CE"/>
+<wire x1="91.44" y1="-81.28" x2="68.58" y2="-81.28" width="0.1524" layer="91"/>
+<label x="76.2" y="-81.28" size="1.778" layer="95"/>
+</segment>
+<segment>
+<pinref part="U$1" gate="G$1" pin="27"/>
+<wire x1="58.42" y1="-2.54" x2="33.02" y2="-2.54" width="0.1524" layer="91"/>
+</segment>
+</net>
